Commit message: Modified transforms

File: cartographer_ros/urdf/G22_microstrainIMU.urdf (robot description, URDF)
Before this commit: robot cartographer_backpack_3d, 3 links, 2 joints
Joints:
- joint imu_link_joint: origin xyz=0 0 0 rpy=3.1416 0 0 -> xyz=0 -0.14 0 rpy=3.1416 0 0
- joint os1_link_joint: origin xyz=-0.267 0 0.08 rpy=0 0 3.1416 -> xyz=-0.127 0 0.08 rpy=0 0 3.1416

Commit message: Tuned parameters on desktop NUC, slightly better, but still some drift when turning

File: cartographer_ros/urdf/G22_microstrainIMU.urdf (robot description, URDF)
Before this commit: robot cartographer_backpack_3d, 3 links, 2 joints
Joints:
- joint imu_link_joint: origin xyz=0 -0.14 0 rpy=3.1416 0 0 -> xyz=-0.14 0 0 rpy=0 -3.14 -1.57
- joint os1_link_joint: origin xyz=-0.127 0 0.08 rpy=0 0 3.1416 -> xyz=0.127 0 0.08 rpy=0 0 0

Commit message: tuned IMU transform based on map drift

File: cartographer_ros/urdf/G22_microstrainIMU.urdf (robot description, URDF)
Before this commit: robot cartographer_backpack_3d, 3 links, 2 joints
Joints:
- joint imu_link_joint: origin xyz=-0.14 0 0 rpy=0 -3.14 -1.57 -> xyz=-0.14 0 0 rpy=0 -3.24 -1.55

Commit message: Configuration used to get good results at Capital Prize Mine Testing on 7/21/2019. Low drift and fast loop closures. No odometry used. Full 360 degree FOV of Ouster and IMU.

File: cartographer_ros/urdf/G22_microstrainIMU.urdf (robot description, URDF)
Before this commit: robot cartographer_backpack_3d, 3 links, 2 joints
Links:
- added link laser; visual cylinder length=0.02 radius=0.03
Joints:
- added joint rplidar_link_joint: type fixed, parent base_link, child laser, origin xyz=0.267 0 0.12 rpy=0 0 0
- joint imu_link_joint: origin xyz=-0.14 0 0 rpy=0 -3.24 -1.55 -> xyz=0 0 0 rpy=0 -3.14 -1.57
- joint os1_link_joint: origin xyz=0.127 0 0.08 rpy=0 0 0 -> xyz=0.267 0 0.08 rpy=0 0 0
