Commit message: Updated cartographer transforms, note that I had to set 3dm_gx5_15 (0 0 0) relative to base_link frame.

File: cartographer_ros/urdf/H02_microstrainIMU.urdf (robot description, URDF)
Before this commit: robot cartographer_backpack_3d, 4 links, 3 joints
Links:
- removed link os1
- added link os1_sensor; visual cylinder length=0.07 radius=0.05
Joints:
- joint os1_link_joint: child os1 -> os1_sensor; origin xyz=0.267 0 0.08 rpy=0 0 0 -> xyz=0 0 0.70 rpy=0 0 0

Commit message: Fixed transform, tracking imu frame now, but the map frame is yawed incorrectly. When fusing in odometry to cartographer, will have to change the tracking frame to base_link and set the imu to base link transform to (0 0 0).

File: cartographer_ros/urdf/H02_microstrainIMU.urdf (robot description, URDF)
Before this commit: robot cartographer_backpack_3d, 4 links, 3 joints
Links:
- removed link laser
Joints:
- removed joint rplidar_link_joint
- joint imu_link_joint: origin xyz=0 0 0 rpy=0 -3.14 -1.57 -> xyz=0 -0.020 0.630 rpy=3.14 0 1.57

Commit message: Updated to 2D cartographer.

File: cartographer_ros/urdf/H02_microstrainIMU.urdf (robot description, URDF)
Before this commit: robot cartographer_backpack_3d, 3 links, 2 joints
Joints:
- joint imu_link_joint: origin xyz=0 -0.020 0.630 rpy=3.14 0 1.57 -> xyz=0 0 0 rpy=3.14 0 1.57
